Commit message: Update myrobot.urdf

File: phobosexp/nazifbot/urdf/myrobot.urdf (robot description, URDF)
Before this commit: robot nazifbot, 6 links, 5 joints
Links:
- link chasis_link: geometry collision box size=15.77345 13.32786 14.73515; visual mesh filename=package://my_robot/meshes/dae/NEW DESIGN Straight.dae scale=0.02663 0.02663 0.02663
- link obj8.004_link: geometry collision box size=5.94552 1.39047 1.25234; visual mesh filename=package://my_robot/meshes/dae/obj8.004.dae scale=-0.04184 -0.04184 -0.04184
- link wheel_front_left_link: geometry collision cylinder length=1.58747 radius=1.58749; visual mesh filename=package://my_robot/meshes/dae/wheel_front_left.dae scale=28.03236 28.03236 28.03236
- link wheel_front_right_link: geometry collision cylinder length=1.58747 radius=1.58749; visual mesh filename=package://my_robot/meshes/dae/wheel_front_right.dae scale=28.03236 28.03236 28.03236
- link wheel_rear_left_link: geometry collision cylinder length=1.58747 radius=1.58747; visual mesh filename=package://my_robot/meshes/dae/wheel_rear_left.dae scale=28.03236 28.03236 28.03236
- link wheel_rear_right_link: geometry collision cylinder length=1.58750 radius=1.58747; visual mesh filename=package://my_robot/meshes/dae/wheel_rear_right.001.dae scale=28.03236 28.03236 28.03236
