Commit message: Added a README, CMakeLists.txt, a launch file.

File: urdf/my_robot.urdf (robot description, URDF)
Before this commit: robot my_robot, 6 links, 5 joints
Links:
- link base_link: geometry collision mesh filename=package://my_robot/meshes/chassis.dae scale=0.3 0.3 0.3; visual mesh filename=package://my_robot/meshes/chassis.dae scale=0.3 0.3 0.3
- link realsense_link: geometry collision mesh filename=package://my_robot/meshes/realsense.dae scale=0.1 0.1 0.1; visual mesh filename=package://my_robot/meshes/realsense.dae scale=0.1 0.1 0.1
- link wheel_front_left: geometry collision mesh filename=package://my_robot/meshes/wheel_front_left.dae scale=0.3 0.3 0.3; visual mesh filename=package://my_robot/meshes/wheel_front_left.dae scale=0.3 0.3 0.3
- link wheel_front_right: geometry collision mesh filename=package://my_robot/meshes/wheel_front_right.dae scale=0.3 0.3 0.3; visual mesh filename=package://my_robot/meshes/wheel_front_right.dae scale=0.3 0.3 0.3
- link wheel_rear_left: geometry collision mesh filename=package://my_robot/meshes/wheel_rear_left.dae scale=0.3 0.3 0.3; visual mesh filename=package://my_robot/meshes/wheel_rear_left.dae scale=0.3 0.3 0.3
- link wheel_rear_right: geometry collision mesh filename=package://my_robot/meshes/wheel_rear_right.dae scale=0.3 0.3 0.3; visual mesh filename=package://my_robot/meshes/wheel_rear_right.dae scale=0.3 0.3 0.3

Commit message: Update my_robot.urdf

File: urdf/my_robot.urdf (robot description, URDF)
Before this commit: robot my_robot, 6 links, 5 joints
Links:
- removed link base_link
- removed link realsense_link
- removed link wheel_front_left
- removed link wheel_front_right
- removed link wheel_rear_left
- removed link wheel_rear_right
- added link chasis_link, mass 7.32100; collision box size=15.77345 13.32786 14.73515; visual mesh filename=package://my_robot/meshes/dae/NEW DESIGN Straight.dae scale=0.02663 0.02663 0.02663
- added link obj8.004_link, mass 1.44100; collision box size=5.94552 1.39047 1.25234; visual mesh filename=package://my_robot/meshes/dae/obj8.004.dae scale=-0.04184 -0.04184 -0.04184
- added link wheel_front_left_link, mass 2.58100; collision cylinder length=1.58747 radius=1.58749; visual mesh filename=package://my_robot/meshes/dae/wheel_front_left.dae scale=28.03236 28.03236 28.03236
- added link wheel_front_right_link, mass 2.58100; collision cylinder length=1.58747 radius=1.58749; visual mesh filename=package://my_robot/meshes/dae/wheel_front_right.dae scale=28.03236 28.03236 28.03236
- added link wheel_rear_left_link, mass 2.58100; collision cylinder length=1.58747 radius=1.58747; visual mesh filename=package://my_robot/meshes/dae/wheel_rear_left.dae scale=28.03236 28.03236 28.03236
- added link wheel_rear_right_link, mass 2.58100; collision cylinder length=1.58750 radius=1.58747; visual mesh filename=package://my_robot/meshes/dae/wheel_rear_right.001.dae scale=28.03236 28.03236 28.03236
Joints:
- removed joint joint_realsense
- removed joint joint_wheel_front_left
- removed joint joint_wheel_front_right
- removed joint joint_wheel_rear_left
- removed joint joint_wheel_rear_right
- added joint obj8.004_link_joint: type fixed, parent chasis_link, child obj8.004_link, origin xyz=7.54713 0.00000 10.52073 rpy=0.00000 0.00000 1.57080
- added joint wheel_front_left_link_joint: type continuous, parent chasis_link, child wheel_front_left_link, origin xyz=6.13767 -8.60360 -5.95609 rpy=1.57080 0.00000 0.00000, axis 0.00000 0.00000 1.00000, limit lower=0 upper=0 effort=9.99000 velocity=10.44000
- added joint wheel_front_right_link_joint: type continuous, parent chasis_link, child wheel_front_right_link, origin xyz=6.13766 8.43827 -5.95614 rpy=1.57080 0.00000 0.00000, axis 0.00000 0.00000 1.00000, limit lower=0 upper=0 effort=9.99000 velocity=10.44000
- added joint wheel_rear_left_link_joint: type continuous, parent chasis_link, child wheel_rear_left_link, origin xyz=-9.19146 -8.60328 -5.95606 rpy=1.57080 0.00000 0.00000, axis 0.00000 0.00000 1.00000, limit lower=0 upper=0 effort=9.99000 velocity=10.44000
- added joint wheel_rear_right_link_joint: type continuous, parent chasis_link, child wheel_rear_right_link, origin xyz=-9.19136 8.43863 -5.95615 rpy=1.57080 0.00000 0.00000, axis 0.00000 0.00000 1.00000, limit lower=0 upper=0 effort=9.99000 velocity=10.44000
